Commit message: V3 URDF integration: replace old assembly with SolidWorks V3 5-bar linkage
- Replace URDF with V3 SolidWorks export (5 joints, 6 links, no trays)
- Add V3 mesh STLs (base_link, Link_1-4, Endeffector)
- Update IK node: V3 joint names, correct IK-to-URDF mapping (no yaw double-count)
- Remove startup home seeding — publish zeros until first /ik_target
- Update arduino_bridge and mks_servo42c_bridge with V3 joint names
- Update launch file: world->base_link static TF

File: Main_Assembly_1/urdf/Main_Assembly_1.urdf (robot description, URDF)
Before this commit: robot Main_Assembly_1, 11 links, 10 joints
Links:
- removed link Front_tray
- removed link Tray_left
- removed link channel_suction_link
- removed link gear_suction
- removed link link_left
- removed link motor_Link_right
- removed link motor_link_left
- removed link right_link
- removed link suction_link
- removed link tray_base_link
- added link Endeffector, mass 0.0288633825048563; collision mesh filename=package://Main_Assembly_1/meshes/Endeffector.STL; visual mesh filename=package://Main_Assembly_1/meshes/Endeffector.STL
- added link Link_1, mass 0.10866; collision mesh filename=package://Main_Assembly_1/meshes/Link_1.STL; visual mesh filename=package://Main_Assembly_1/meshes/Link_1.STL
- added link Link_2, mass 0.108656751757487; collision mesh filename=package://Main_Assembly_1/meshes/Link_2.STL; visual mesh filename=package://Main_Assembly_1/meshes/Link_2.STL
- added link Link_3, mass 0.107515397534699; collision mesh filename=package://Main_Assembly_1/meshes/Link_3.STL; visual mesh filename=package://Main_Assembly_1/meshes/Link_3.STL
- added link Link_4, mass 0.0932618314359105; collision mesh filename=package://Main_Assembly_1/meshes/Link_4.STL; visual mesh filename=package://Main_Assembly_1/meshes/Link_4.STL
- link base_link: mass 0.289654091949094 -> 0.965408329881284
Joints:
- removed joint Front_tray_joint
- removed joint Left_Tray_joint
- removed joint gear_servo_suction_joint
- removed joint joint_link_left
- removed joint motor_joint_left
- removed joint motor_joint_right
- removed joint right_joint_link
- removed joint suction_channel
- removed joint suction_joint_link
- removed joint tray_to_linkage_joint
- added joint Joint_1: type revolute, parent base_link, child Link_1, origin xyz=0.22303 -0.17462 0.12681 rpy=-1.5853 -0.016051 -0.40717, axis 0 1 0, limit lower=-3.14159 upper=3.14159 effort=10 velocity=3.14
- added joint Joint_2: type revolute, parent base_link, child Link_2, origin xyz=0.033931 -0.17377 0.1045 rpy=-1.5924 -0.0012905 0.37069, axis 0 1 0, limit lower=-3.14159 upper=3.14159 effort=10 velocity=3.14
- added joint Joint_3: type revolute, parent Link_1, child Link_3, origin xyz=0 0 0.2 rpy=0 0.15538 0, axis 0 1 0, limit lower=-3.14159 upper=3.14159 effort=10 velocity=3.14
- added joint Joint_4: type revolute, parent Link_2, child Link_4, origin xyz=0 -0.0036364 0.2 rpy=0 0.16756 -3.1416, axis 0 1 0, limit lower=-3.14159 upper=3.14159 effort=10 velocity=3.14
- added joint Joint_5: type revolute, parent Link_3, child Endeffector, origin xyz=-0.2 -0.0063467 -0.00014871 rpy=-3.1416 -1.5579 0, axis 0 1 0, limit lower=-3.14159 upper=3.14159 effort=10 velocity=3.14
